Commit message: add rviz launch ans setup mov base library

File: valrob_description/urdf/valrob_description.urdf.xacro (robot description, xacro)
@@ -118,5 +118,5 @@
     <inertial>
       <origin
-        xyz="9.71445146547012E-16 -0.0150000000000003 9.43689570931383E-16"
+        xyz="0 0 0.015"
         rpy="0 0 0" />
       <mass value="0.19085175370558" />
@@ -130,5 +130,5 @@
     </inertial>
     <visual>
-      <origin xyz="0 0 0" rpy="0 0 0" />
+      <origin xyz="0 0 0" rpy="1.57 0 0" />
       <geometry>
         <mesh filename="package://valrob_description/meshes/laser.STL" />
@@ -137,5 +137,5 @@
     </visual>
     <collision>
-      <origin xyz="0 0 0" rpy="0 0 0" />
+      <origin xyz="0 0 0" rpy="1.57 0 0" />
       <geometry>
         <mesh filename="package://valrob_description/meshes/laser.STL" />
@@ -147,8 +147,8 @@
     <origin
       xyz="0 0 0.388"
-      rpy="-1.5708 0 3.1416" />
+      rpy="0 0 0" />
     <parent link="base_link" />
     <child link="laser" />
-    <axis xyz="0 1 0" />
+    <axis xyz="0 0 0" />
   </joint>
   <!-- imu -->
